File: display/display.kicad_pcb (KiCad board)
At the start: 2 copper layers, 55 x 29.5 mm, 20 parts, among them J1 Conn, J2 Conn_01x02_Male, M1 MountingHole_2.2mm_M2, M3 MountingHole_2.2mm_M2, M4 display_cutout, U1 MAN74A, U2 MAN74A, U3 AS1115-BSST, U4 MAN74A, U5 MAN74A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

Commit message: Added initial code base, improved and fixed hardware up to Rev 1.5/1.2 for the main and display boards respectively, and add pictures of (mostly) complete result
Parts:
- J1: footprint personal:DISPIO10 -> Connector_PinHeader_2.54mm:PinHeader_2x05_P2.54mm_Horizontal
- J2: value Conn_01x02_Male -> KEYAB
- JP1: value SolderJumper_3_Bridged123 -> KEY_EN
- R_ISET1, R_ISET2: value 47k -> 43k
- moved J1 10.5 mm to (100.8, 75.7), turned to 90 degrees
Connections:
- C1 pad 2: +5VD -> VCC
- C4 pad 1: +5VD -> VCC
- J1 pad 1: +5VD -> GND
- J1 pad 10: GND -> VCC
- J1 pad 2: +5VD -> GND
- J1 pad 3: Net-(J1-Pad3) -> Net-(R3-Pad2)
- J1 pad 4: Net-(J1-Pad3) -> Net-(R3-Pad2)
- J1 pad 7: Net-(J1-Pad7) -> Net-(R1-Pad2)
- J1 pad 8: Net-(J1-Pad7) -> Net-(R1-Pad2)
- J1 pad 9: GND -> VCC
- R1 pad 1: +5VD -> VCC
- R1 pad 2: Net-(J1-Pad3) -> Net-(R1-Pad2)
- R2 pad 1: +5VD -> VCC
- R3 pad 1: +5VD -> VCC
- R3 pad 2: Net-(J1-Pad7) -> Net-(R3-Pad2)
- R_TRIM1 pad 2: +5VD -> VCC
- U3 pad 14: Net-(J1-Pad3) -> Net-(R1-Pad2)
- U3 pad 19: +5VD -> VCC
- U3 pad 24: Net-(J1-Pad7) -> Net-(R3-Pad2)
Routing:
- net VCC: track 0.00 -> 112.1 mm
- net +5VD: track 112.1 -> 0.00 mm
- net Net-(R1-Pad2): track 0.00 -> 29.3 mm, vias 0 -> 1
- net Net-(J1-Pad3): track 29.3 -> 0.00 mm, vias 1 -> 0
- net Net-(R3-Pad2): track 0.00 -> 17.0 mm, vias 0 -> 1
- net Net-(J1-Pad7): track 17.0 -> 0.00 mm, vias 1 -> 0
Other:
- board text added: "2022 REV. 1.2 JZACT"
- board text removed: "2022 REV. 1.1 JZACT"
