File: main_board/main_board.kicad_pcb (KiCad board)
At the start: 2 copper layers, 85 x 94.5 mm, 81 parts, among them J1 Screw_Terminal_01x03, J2 Conn, J3 Screw_Terminal_01x02, J4 Screw_Terminal_01x02, J5 SPI, J6 UPDI, J7 EARTH JUMPER, SW1 RESET, SW2 DISP. MODE, U1 25LC640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

Commit message: Added initial code base, improved and fixed hardware up to Rev 1.5/1.2 for the main and display boards respectively, and add pictures of (mostly) complete result
Parts:
- removed D6: M4, Diode_SMD:D_SMB
- removed F1: PTSA080515V012, Fuse:Fuse_0805_2012Metric_Pad1.15x1.40mm_HandSolder
- F2, F3: value 1.25A -> 5A Slow
- J2: footprint personal:DISPIO10 -> Connector_PinHeader_2.54mm:PinHeader_2x05_P2.54mm_Vertical
- J7: footprint Connector_PinSocket_2.54mm:PinSocket_1x01_P2.54mm_Vertical -> Connector_PinHeader_2.54mm:PinHeader_1x01_P2.54mm_Vertical
- SW2: footprint Connector_PinSocket_2.54mm:PinSocket_1x02_P2.54mm_Vertical -> Connector_PinHeader_2.54mm:PinHeader_1x02_P2.54mm_Vertical
- turned C13 to 180 degrees
- turned R3 to 0 degrees
Connections:
- C13 pad 1: Net-(C13-Pad1) -> Net-(R3-Pad1)
- FB1 pad 2: Net-(F1-Pad1) -> Net-(C17-Pad1)
- SW1 pad 1: Net-(C13-Pad1) -> GND
Routing:
- net 5_Out: track 50.2 -> 33.0 mm, vias 16 -> 8
- net Net-(C15-Pad1): track 17.3 -> 12.3 mm
- net Net-(C13-Pad1): track 3.50 -> 0.00 mm
- net GND: track 158.1 -> 161.4 mm
- net Net-(R3-Pad1): track 3.51 -> 6.60 mm
- net Net-(F1-Pad1): track 2.17 -> 0.00 mm
- net ~{RESET}: track 26.5 -> 27.8 mm
- net Net-(C17-Pad1): track 15.4 -> 14.7 mm
Other:
- board text added: "2022 REV. 1.5 JZACT"
- board text removed: "2022 REV. 1.4 JZACT"
